File: microcontrollerCarriers/Poseidon-Pico/Poseidon-Pico.kicad_pcb (KiCad board)
At the start: 2 copper layers, 61.8 x 70.8 mm, 61 parts, among them J1 Conn_01x03, J10 Conn_01x03, J11 Conn_01x03, J12 Conn_01x03, J13 Conn_01x03, J14 Conn_01x03, J15 Conn_01x03, J16 Conn_01x04, J17 Conn_01x02, J18 Conn_01x04, J2 Conn_01x03, J3 Conn_01x03, J4 Conn_01x03, J5 Conn_01x03, J6 Conn_01x03, J7 Conn_01x03, J8 Conn_01x03, J9 Conn_01x03, U1 Pico, U2 LM4040DBZ-3, U3 TXB0108DQSR, U5 NCP1117-5.0_SOT223, U7 MCP2517FD-xSL, U8 MCP2542FDxMF, Y1 40 MHz 9 pF

Commit message: Fix JST-SH 3d model and pins, add silkscreen to Pico
Parts:
- C9: renamed from C4; value 10 uF -> 10 uF 35v
- turned J8 to 90 degrees
- renumbered C2 to C1, C1 to C2, C13 to C3, C12 to C4, C8 to C5, C11 to C6, C3 to C8, D4 to D3, D3 to D4, J11 to J1, J14 to J10, J7 to J11, J13 to J12, J2 to J13, J15 to J14, J3 to J15, J12 to J16, J6 to J2, J10 to J3, J5 to J4, J9 to J5, J4 to J6, J8 to J7, J16 to J8, J1 to J9, R6 to R1, R17 to R10, R10 to R12, R15 to R13, R20 to R14, R19 to R15, R4 to R2, R7 to R3, R2 to R4, R1 to R5, R8 to R6, R12 to R7, R3 to R8, R5 to R9, U2 to U1, U3 to U2, U1 to U3, U8 to U4, U7 to U5, U5 to U6
Connections:
- net GPIO19 renamed GPIO8
- net GPIO20 renamed GPIO9
- net GPIO21 renamed GPIO10
- net GPIO22 renamed GPIO11
- J8 pad 1: SCL -> GND
- J8 pad 2: SDA -> Net-(D2-K)
- J8 pad 3: Net-(D2-K) -> SDA
- J8 pad 4: GND -> SCL
Routing:
- net SCL: track 40.1 -> 43.2 mm
- net SDA: track 44.8 -> 47.5 mm
- net Net-(D2-K): track 2.14 -> 4.79 mm
- net +3.3V: track 139.6 -> 142.1 mm
- net GND: track 38.8 -> 38.1 mm
Other:
- board text added: "3.3V"
- board text added: "5v"
- board text added: "6.5V < VIN < 20V"
- board text added: "A0"
- board text added: "A1"
- board text added: "A2"
- board text added: "Bridge to terminate CAN"
- board text added: "D0"
- board text added: "D1"
- board text added: "D10"
- board text added: "D11"
- board text added: "D12"
- board text added: "D2"
- board text added: "D3"
- board text added: "D4"
- board text added: "D5"
- board text added: "D6"
- board text added: "D7"
- board text added: "D8"
- board text added: "D9"
- board text added: "GND"
- board text added: "H"
- board text added: "H = YLW L = GRN"
- board text added: "L"
- board text added: "VIN"
