File: microcontrollerCarriers/Poseidon-Pico/Poseidon-Pico.kicad_sch (KiCad schematic)
At the start: 55 parts, among them J1 Conn_01x03, J10 Conn_01x03, J11 Conn_01x03, J12 Conn_01x03, J13 Conn_01x03, J14 Conn_01x03, J15 Conn_01x03, J16 Conn_01x04, J17 Conn_01x02, J18 Conn_01x04, J2 Conn_01x03, J3 Conn_01x03, J4 Conn_01x03, J5 Conn_01x03, J6 Conn_01x03, J7 Conn_01x03, J8 Conn_01x03, J9 Conn_01x03, U1 Pico, U2 LM4040DBZ-3, U2 MCP2542FDxMF, U3 TXB0108DQSR, U5 MCP2517FD-xSL, U5 NCP1117-5.0_SOT223, Y1 40 MHz 9 pF

Commit message: Fix JST-SH 3d model and pins, add silkscreen to Pico
Parts:
- C9: renamed from C4; value 10 uF -> 10 uF 35v
- renumbered C2 to C1, C1 to C2, C3 to C8, D4 to D3, D3 to D4, J11 to J1, J14 to J10, J7 to J11, J13 to J12, J2 to J13, J15 to J14, J3 to J15, J12 to J16, J6 to J2, J10 to J3, J5 to J4, J9 to J5, J4 to J6, J8 to J7, J16 to J8, J1 to J9, R6 to R1, R17 to R10, R10 to R12, R15 to R13, R4 to R2, R7 to R3, R2 to R4, R1 to R5, R8 to R6, R12 to R7, R3 to R8, R5 to R9, U2 to U1, U3 to U2, U1 to U3, U5 to U6
Connections:
- net GND: now also J8.1 (Pin_1); no longer J8.4 (Pin_4)
- net SCL: now also J8.4 (Pin_4); no longer J8.1 (Pin_1)
- net SDA: now also J8.3 (Pin_3); no longer J8.2 (Pin_2)
- net at D2.1 (K): now also J8.2 (Pin_2); no longer J8.3 (Pin_3)
- net GPIO19 renamed GPIO8
- net GPIO20 renamed GPIO9
- net GPIO21 renamed GPIO10
- net GPIO22 renamed GPIO11
Other:
- note added: "CAN Transciever, Controller, Connector, and Optional Termination"
- note removed: "CAN Controller & Transciever"
- note removed: "CAN Transciever & Connector"
- moved on the sheet: C2, C3, C4, C6, C8, C9, D1, D2, D4, J17, J18, J2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
