File: microcontrollerCarriers/Poseidon-Teensy/Poseidon-Teensy.kicad_pcb (KiCad board)
At the start: 4 copper layers, 61.8 x 70.8 mm, 52 parts, among them J1 Conn_01x03, J10 Conn_01x03, J11 Conn_01x03, J12 Conn_01x03, J13 Conn_01x03, J14 Conn_01x03, J15 Conn_01x03, J16 Conn_01x04, J19 Conn_01x02, J2 Conn_01x03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

Commit message: Fix JST-SH 3d model and pins, add silkscreen to Pico
Parts:
- turned J16 to 90 degrees
Connections:
- J16 pad 1: SCL -> GND
- J16 pad 2: SDA -> Net-(D2-K)
- J16 pad 3: Net-(D2-K) -> SDA
- J16 pad 4: GND -> SCL
Routing:
- net SCL: track 24.1 -> 27.3 mm
- net GND: track 28.9 -> 31.7 mm
- net SDA: track 21.7 -> 24.4 mm
- net Net-(D2-K): track 2.10 -> 4.75 mm
Other:
- board text removed: "SCL"
- board text removed: "SDA"
