File: Hephaestos/Hephaestos.kicad_pcb (KiCad board)
At the start: 4 copper layers, 106.8 x 61 mm, 154 parts, among them J1 Conn_01x02, J10 Conn_01x02, J11 Conn_01x02, J2 Conn_01x02, J3 Conn_01x02, J4 Conn_01x02, J5 Conn_02x05_Counter_Clockwise, J6 Conn_01x02, J7 Conn_01x04, J8 Conn_01x02, J9 Conn_01x02, Q1 CSD17577Q5A, Q2 CSD17577Q5A, U1 MCP6001-OT, U10 MCP6001-OT, U11 MCP6001-OT, U12 MCP6001-OT, U13 STM32F042C6Tx, U2 MCP6001-OT, U3 MCP6001-OT, U4 MCP6001-OT, U5 AP2205K-3.3, U8 SN65HVD232, U9 MCP6001-OT, Y1 16 MHz 9 pF

Commit message: Add second bulk cap
Parts:
- added C17: 100 uF 35v, Capacitor_SMD:CP_Elec_6.3x7.7, F.Cu at (207.7, 103.0)
- moved 1 53.3 mm to (156.0, 95.8)
- moved 2 53.3 mm to (156.1, 95.8)
- renumbered C12 to C10, C15 to C11, C28 to C12, C17 to C13, C18 to C14, C19 to C15, C20 to C16, C21 to C18, C5 to C19, C24 to C20, C25 to C21, C26 to C22, C27 to C23, C6 to C5, C7 to C6, C8 to C7, C9 to C8, C11 to C9, R70 to R26, R26 to R27, R27 to R28, R28 to R29, R29 to R30, R30 to R31, R31 to R32, R32 to R33, R33 to R34, R34 to R35, R37 to R36, R71 to R37, R43 to R41, R44 to R42, R69 to R43, R45 to R44, R46 to R45, R47 to R46, R48 to R47, R49 to R48, R50 to R49, R51 to R50, R52 to R51, R53 to R52, R54 to R53, R55 to R54, R56 to R55, R57 to R56, R58 to R57, R59 to R58, R60 to R59, R61 to R60, R62 to R61, R63 to R62, R64 to R63, R65 to R64, R66 to R65, R67 to R66, R68 to R67, U11 to U10, U12 to U11, U13 to U6, U8 to U7, U9 to U8, U10 to U9
Routing:
- net ADC_THERM: track 14.7 -> 11.1 mm, vias 2 -> 0
- net ADC_VCCDIV: track 12.8 -> 10.0 mm, vias 2 -> 0
- net GND: track 131.7 -> 134.2 mm, vias 53 -> 54
